File: simpleton.kicad_pcb (KiCad board)
At the start: 2 copper layers, 273 x 123.9 mm, 73 parts, among them U1 blackpill

Commit message: namtab.
Other:
- board size 273 x 123.9 mm -> 271.3 x 124.9 mm

Commit message: ground.
Connections:
- U1 pad 19: (no net) -> GND
- U1 pad 39: (no net) -> GND
Routing:
- added copper zone on B.Cu, net GND
- added copper zone on F.Cu, net GND
- removed copper zone on B.Cu, net (none)
- removed copper zone on F.Cu, net (none)
