File: simpleton.sch (KiCad schematic (older format))
At the start: 73 parts, among them U1 blackpill

Commit message: ground.
Connections:
- net GND: now reaches U1.19 (PG)
- net GND: now also U1.39 (PG)
Changed lines of the file:
@@
 Text GLabel 4850 6450 0    50   Input ~ 0
 COL4
+Text GLabel 5850 4950 2    50   Input ~ 0
+GND
+Text GLabel 4850 6650 0    50   Input ~ 0
+GND
 $EndSCHEMATC
